File: Flyback_STD.kicad_pcb (KiCad board)
At the start: 2 copper layers, 60.6 x 27.5 mm, 104 parts, among them P1 VIN, P2 GND, P3 VOUT, P4 PGND, Q1 HY1420C2, Q2 HSBB0012, U1 VPC2188B

Commit message: Update Coil
Parts:
- added REF**: NPTH-C_0805, 302_MECH_PAD:NPTH-C_0805, F.Cu at (111.4, 106.8)
- added REF**: NPTH-C_0805, 302_MECH_PAD:NPTH-C_0805, F.Cu at (111.4, 107.6)
- added REF**: NPTH-C_0805, 302_MECH_PAD:NPTH-C_0805, F.Cu at (111.4, 106.0)
- added REF**: NPTH-C_0805, 302_MECH_PAD:NPTH-C_0805, F.Cu at (111.4, 108.4)
- REF** (x18): value NPTH-C_1006 -> NPTH-C_0805; footprint 302_MECH_PAD:NPTH-C_1006 -> 302_MECH_PAD:NPTH-C_0805
- moved REF** 3.30 mm to (111.4, 105.2)
- moved REF** 3.10 mm to (111.4, 104.4)
- moved REF** 2.90 mm to (111.4, 103.6)
- moved REF** 2.70 mm to (111.4, 102.8)
- moved REF** 2.50 mm to (111.4, 102.0)
- moved REF** 2.30 mm to (111.4, 101.2)
- moved REF** 2.10 mm to (111.4, 100.4)
- moved REF** 1.90 mm to (111.4, 99.6)
- moved REF** 1.70 mm to (111.4, 98.8)
- moved REF** 1.51 mm to (111.4, 98.0)
- moved REF** 1.31 mm to (111.4, 97.2)
- moved REF** 1.11 mm to (111.4, 96.4)
- moved REF** 0.91 mm to (111.4, 95.6)
- moved REF** 0.71 mm to (111.4, 94.8)
- moved REF** 0.52 mm to (111.4, 94.0)
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Routing:
- net VBUS: track 118.7 -> 179.1 mm, vias 102 -> 109
- net GND: track 111.5 -> 106.8 mm, vias 85 -> 86
- net /CS: track 39.7 -> 37.9 mm
- net GNDPWR: track 70.6 -> 70.2 mm, vias 68 -> 69
Other:
- outline, holes or cut-outs redrawn

Commit message: Daily update
Routing:
- net VBUS: track 179.1 -> 60.4 mm, vias 109 -> 97
- net GND: track 106.8 -> 107.7 mm
- net /CS: track 37.9 -> 37.1 mm
Other:
- board size 60.6 x 27.5 mm -> 60.8 x 27.5 mm
- board text added: "v0.9.2"
- board text removed: "v0.9.1"

Commit message: Remake project
Parts:
- removed C1, C2: 100nF, 001_GN_RCL_SMD:C0603(1608M)
- removed C10: 10uF, 001_GN_RCL_SMD:C0805(2012M)
- removed C11: 120uF, 007_GN_POLAR-CAP_SMD:CL-0608
- removed C12, C13, C14, C15, C16, C17, C18, C19: 10uF, 001_GN_RCL_SMD:C0603(1608M)
- removed C3: 1nF, 001_GN_RCL_SMD:C0603(1608M)
- removed C4, C5, C6, C7: 4.7uF, 001_GN_RCL_SMD:C1210(3225M)
- removed C8: 100uF, 007_GN_POLAR-CAP_SMD:CL-1010
- removed C9: 1nF, 001_GN_RCL_SMD:C0805(2012M)
- removed D1, D4: DS110W, 002_GN_TWO-PIN_PLASTIC_SMD:SOD-123F
- removed D2, D3: DS120W, 002_GN_TWO-PIN_PLASTIC_SMD:SOD-123F
- removed D5, D6: SB2080L, 102_SP_POWER_DIODE_SMD:TO-277B
- removed L1: 10uH, 008_GN_POWER-CHOKE_SMD:MC-2520
- removed Q1: HY1420C2, 103_SP_POWER_TRANSISTOR_SMD:SON-FET_6050
- removed Q2: HSBB0012, 103_SP_POWER_TRANSISTOR_SMD:SON-FET_3333
- removed R1: 100R, 001_GN_RCL_SMD:R0603(1608M)
- removed R10: 3.9k, 001_GN_RCL_SMD:R0603(1608M)
- removed R11: 2.2k, 001_GN_RCL_SMD:R1206(3216M)
- removed R2: 100k, 001_GN_RCL_SMD:R0603(1608M)
- removed R3: 5.6k, 001_GN_RCL_SMD:R0603(1608M)
- removed R4: 27k, 001_GN_RCL_SMD:R0603(1608M)
- removed R5: RL1210A680K, 001_GN_RCL_SMD:R1210(3225M)
- removed R6: 2.2R, 001_GN_RCL_SMD:R0603(1608M)
- removed R7: 10k, 001_GN_RCL_SMD:R0603(1608M)
- removed R8: 25mR/1W, 001_GN_RCL_SMD:R1206(3216M)
- removed R9: 33k, 001_GN_RCL_SMD:R0603(1608M)
- removed REF** (x22): NPTH-C_0805, 302_MECH_PAD:NPTH-C_0805
- removed REF** (x42): SMP-C_15, 302_MECH_PAD:SMP-C_15
- removed U1: VPC2188B, 004_GN_MIDDLE-SEMI_SMD:MSOP-10_3030
Routing:
- net GND: track 107.7 -> 52.2 mm, vias 86 -> 2
- net VBUS: track 60.4 -> 109.2 mm, vias 97 -> 17
- net VDD: track 43.5 -> 0.00 mm, vias 3 -> 0
- net /CS: track 37.1 -> 0.00 mm, vias 5 -> 0
- net GNDPWR: track 70.2 -> 53.2 mm, vias 69 -> 5
- net /GT_U: track 16.3 -> 0.00 mm, vias 3 -> 0
- net Vdrive: track 5.48 -> 0.00 mm
- net /UVP: track 5.33 -> 0.00 mm
- net Net-(D2-Anode): track 4.19 -> 0.00 mm
- net Net-(U1-FB): track 3.53 -> 0.00 mm
- net /GT: track 3.27 -> 0.00 mm
- net Net-(D3-Anode): track 2.19 -> 0.00 mm
- net /RT: track 1.61 -> 0.00 mm
- net /SS: track 1.52 -> 0.00 mm
- net Net-(D1-Anode): track 1.38 -> 0.00 mm
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- removed copper zone on F.Cu, net /CS
- removed copper zone on B.Cu, net GND
- removed copper zone on F.Cu, net GND
- removed copper zone on B.Cu, net GNDPWR
- removed copper zone on F.Cu, net GNDPWR
- removed copper zone on B.Cu, net VBUS
- removed copper zone on F.Cu, net VBUS
- removed copper zone on B.Cu, net VDC
- removed copper zone on F.Cu, net VDC
Other:
- board size 60.8 x 27.5 mm -> 22.4 x 27.5 mm
- board text added: "v0.9.1"
- board text removed: "PkgLAN"
- board text removed: "v0.9.2"
