File: Flyback_STD.kicad_sch (KiCad schematic)
At the start: 46 parts, among them P1 BATT+, P2 BATT-, P3 VBUS, P4 GND, Q1 5N20A, T1 TRF-6, U1 OB2106MP, U2 VPC2188B, U4 TL431

Commit message: Daily update
Parts:
- removed C1: 1uF, 001_GN_RCL_SMD:C1206(3216M), symbol 001_Basic_PassiveComponents:101_Capacitor
- removed C10: 220pF, 001_GN_RCL_SMD:C1206(3216M), symbol 001_Basic_PassiveComponents:101_Capacitor
- removed C5: 100nF, 001_GN_RCL_SMD:C0603(1608M), symbol 001_Basic_PassiveComponents:101_Capacitor
- removed C6: 10uF, 001_GN_RCL_SMD:C0805(2012M), symbol 001_Basic_PassiveComponents:101_Capacitor
- removed C7: 1uF, 001_GN_RCL_SMD:C0805(2012M), symbol 001_Basic_PassiveComponents:101_Capacitor
- removed C8: 1uF, 001_GN_RCL_SMD:C2220(5650M), symbol 001_Basic_PassiveComponents:101_Capacitor
- removed C9: 10nF, 001_GN_RCL_SMD:C0603(1608M), symbol 001_Basic_PassiveComponents:101_Capacitor
- removed D2: US1MF, 002_GN_TWO-PIN_PLASTIC_SMD:SMA(DO-214AC), symbol 002_Basic_SingleSemiconductor:001_Diode
- removed D3, D4: DS110W, 002_GN_TWO-PIN_PLASTIC_SMD:SOD-123F, symbol 002_Basic_SingleSemiconductor:002_Diode_Schottky
- removed L1: 100uH, 008_GN_POWER-CHOKE_SMD:MC-0420, symbol 001_Basic_PassiveComponents:202_PowerChoke
- removed PC1: EL817S1(B)(TU)-F, MRLA:OC-4_6546, symbol MRLA:PC-4
- removed R11, R12: 470k, 001_GN_RCL_SMD:R0805(2012M), symbol 001_Basic_PassiveComponents:001_Resistor
- removed R13: 2.2k, 001_GN_RCL_SMD:R0603(1608M), symbol 001_Basic_PassiveComponents:001_Resistor
- removed R19: 5.6k, 001_GN_RCL_SMD:R0603(1608M), symbol 001_Basic_PassiveComponents:001_Resistor
- removed R21: 22R, 001_GN_RCL_SMD:R0603(1608M), symbol 001_Basic_PassiveComponents:001_Resistor
- removed R25, R7, R9: 4.7k, 001_GN_RCL_SMD:R0603(1608M), symbol 001_Basic_PassiveComponents:001_Resistor
- removed R26: 150k, 001_GN_RCL_SMD:R1206(3216M), symbol 001_Basic_PassiveComponents:001_Resistor
- removed R27, R28, R29: 200k, 001_GN_RCL_SMD:R1206(3216M), symbol 001_Basic_PassiveComponents:001_Resistor
- removed R3: 22k, 001_GN_RCL_SMD:R0603(1608M), symbol 001_Basic_PassiveComponents:001_Resistor
- removed R6: 20k, 001_GN_RCL_SMD:R0603(1608M), symbol 001_Basic_PassiveComponents:001_Resistor
- removed T1: TRF-6, MRLA:TRF-6_6P30S, symbol MRLA:TRF-6
- removed U1: OB2106MP, 003_GN_SMALL-SEMI_SMD:SOT-23-6, symbol 204_Power_SMPS-Convertor:OB2106MP
- removed U4: TL431, 003_GN_SMALL-SEMI_SMD:SOT-23, symbol 103_IntegratedCircuit_Reference:TL431
Other:
- note removed: "调试阶段47k"
- moved on the sheet: R14

Commit message: Nightly update
Parts:
- added C1: 10uF, 001_GN_RCL_SMD:C0805(2012M), symbol 001_Basic_PassiveComponents:101_Capacitor
- added C10, C9: 100uF, 007_GN_POLAR-CAP_SMD:CL-1010, symbol 001_Basic_PassiveComponents:102_PolarCapacitor
- added C5, C6, C7, C8: 100uF, 007_GN_POLAR-CAP_SMD:CL-0608, symbol 001_Basic_PassiveComponents:102_PolarCapacitor
- added D2: DS110W, 002_GN_TWO-PIN_PLASTIC_SMD:SOD-123F, symbol 002_Basic_SingleSemiconductor:002_Diode_Schottky
- added D3: SB2080L, 102_SP_POWER_DIODE_SMD:TO-277A, symbol 201_Power_Diode:002_Diode_Schottky
- added R3: 39k, 001_GN_RCL_SMD:R0603(1608M), symbol 001_Basic_PassiveComponents:001_Resistor
- added R6: 3.9k, 001_GN_RCL_SMD:R0603(1608M), symbol 001_Basic_PassiveComponents:001_Resistor
- C4: footprint 001_GN_RCL_SMD:C0603(1608M) -> 001_GN_RCL_SMD:C0805(2012M)
- P1: value BATT+ -> VIN
- P2: value BATT- -> GND
- P3: value VBUS -> VOUT
- P4: value GND -> PGND
- Q1: value 5N20A -> HSBA20N15S; footprint 103_SP_POWER_TRANSISTOR_SMD:TO252-FET_6561 -> 103_SP_POWER_TRANSISTOR_SMD:SON-FET_6050; LCSC (none) -> C701044
- R10: value 80mR/1W -> 30mR/1W; LCSC (none) -> C2988649
- R4: value 22k -> 51k
- R8: value 22R -> 2.2R
Connections:
- net +BATT is gone; now on net VBUS: C4.1, P1.PAD, R1.1, R5.1, U2.2 (Vin)
- net SW_P is gone; now on net VBUS: D1.2 (Anode), Q1.D (Drain)
- net GND: now also C1.2, C10.2, C9.2, D2.2 (Anode), R3.1, R6.2
- net GNDPWR: now also C5.2, C6.2, C7.2, C8.2, D3.A (Anode)
- net VBUS: now also C10.1, C9.1; no longer P3.PAD
- net at U2.10 (FB): now also R3.2, R6.1
- net +10V renamed Vdrive
- net Vdrive: now also C1.1, D2.1 (Cathode)
- net COM: no longer names the net of U2.1 (COM)
- new net VDC: C5.1, C6.1, C7.1, C8.1, D3.K (Cathode), P3.PAD
Other:
- note removed: "调试阶段20k"
- moved on the sheet: C2, C3, C4, D1, P1, P2, P3, P4, Q1, R1, R10, R14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

Commit message: Daily update
Parts:
- removed C10: 100uF, 007_GN_POLAR-CAP_SMD:CL-1010, symbol 001_Basic_PassiveComponents:102_PolarCapacitor
- removed C7, C8: 100uF, 007_GN_POLAR-CAP_SMD:CL-0608, symbol 001_Basic_PassiveComponents:102_PolarCapacitor
- added C7: 100nF, 001_GN_RCL_SMD:C0603(1608M), symbol 001_Basic_PassiveComponents:101_Capacitor
- added D4: SB2080L, 102_SP_POWER_DIODE_SMD:TO-277A, symbol 201_Power_Diode:002_Diode_Schottky
- C2: value 1uF -> 100nF
Connections:
- net GND: now also C7.2
- net GNDPWR: now also D4.A (Anode)
- net VBUS: now also C7.1
- net VDC: now also D4.K (Cathode)

Commit message: Update Flyback_STD.kicad_sch
Parts:
- C4: value 100pF -> 12nF
- D1: value DS110W -> DS120W
- R10: value 30mR/1W -> 25mR/1W
- R2: value 4.7k -> 5.6k
- R3: value 39k -> 36k
- R4: value 51k -> 27k
Changed lines of the file:
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@@
   (symbol (lib_id "002_Basic_SingleSemiconductor:002_Diode_Schottky") (at 119.38 78.74 0) (unit 1)
     (in_bom yes) (on_board yes) (dnp no) (fields_autoplaced)
-    (property "Reference" "D1" (at 119.38 72.39 0)
-      (effects (font (size 1.27 1.27)))
-    )
-    (property "Value" "DS110W" (at 119.38 74.93 0)
+    (property "Reference" "D1" (at 119.38 73.66 0)
+      (effects (font (size 1.27 1.27)))
+    )
+    (property "Value" "DS120W" (at 119.38 76.2 0)
       (effects (font (size 1.27 1.27)))
     )
@@
       (effects (font (size 1.27 1.27)) (justify left))
     )
-    (property "Value" "51k" (at 66.04 113.665 90)
+    (property "Value" "27k" (at 66.04 113.665 90)
       (effects (font (size 1.27 1.27)) (justify left))
     )
@@
   (symbol (lib_id "001_Basic_PassiveComponents:001_Resistor") (at 45.72 111.76 270) (unit 1)
     (in_bom yes) (on_board yes) (dnp no) (fields_autoplaced)
-    (property "Reference" "R2" (at 48.26 110.4899 90)
-      (effects (font (size 1.27 1.27)) (justify left))
-    )
-    (property "Value" "4.7k" (at 48.26 113.0299 90)
+    (property "Reference" "R2" (at 48.26 111.125 90)
+      (effects (font (size 1.27 1.27)) (justify left))
+    )
+    (property "Value" "5.6k" (at 48.26 113.665 90)
       (effects (font (size 1.27 1.27)) (justify left))
     )
@@
       (effects (font (size 1.27 1.27)) (justify left))
     )
-    (property "Value" "39k" (at 147.32 103.505 90)
+    (property "Value" "36k" (at 147.32 103.505 90)
       (effects (font (size 1.27 1.27)) (justify left))
     )
@@
   (symbol (lib_id "001_Basic_PassiveComponents:101_Capacitor") (at 104.14 68.58 0) (unit 1)
     (in_bom yes) (on_board yes) (dnp no) (fields_autoplaced)
-    (property "Reference" "C4" (at 104.14 62.23 0)
-      (effects (font (size 1.27 1.27)))
-    )
-    (property "Value" "100pF" (at 104.14 64.77 0)
+    (property "Reference" "C4" (at 104.14 63.5 0)
+      (effects (font (size 1.27 1.27)))
+    )
+    (property "Value" "12nF" (at 104.14 66.04 0)
       (effects (font (size 1.27 1.27)))
     )
@@
       (effects (font (size 1.27 1.27)) (justify left))
     )
-    (property "Value" "30mR/1W" (at 129.54 118.745 90)
-      (effects (font (size 1.27 1.27)) (justify left))
-    )
+    (property "Value" "25mR/1W" (at 129.54 118.745 90)
+      (effects (font (size 1.27 1.27)) (justify left))
+    )

Commit message: Update to v0.9.1
Parts:
- removed C6: 100uF, 007_GN_POLAR-CAP_SMD:CL-0608, symbol 001_Basic_PassiveComponents:102_PolarCapacitor
- removed R5: 3.3k, 001_GN_RCL_SMD:R1206(3216M), symbol 001_Basic_PassiveComponents:001_Resistor
- added C12, C13, C14, C15, C16, C17, C18, C19: 10uF, 001_GN_RCL_SMD:C0603(1608M), symbol 001_Basic_PassiveComponents:101_Capacitor
- added C4, C5, C6, C7: 4.7uF, 001_GN_RCL_SMD:C1210(3225M), symbol 001_Basic_PassiveComponents:101_Capacitor
- added D1: DS110W, 002_GN_TWO-PIN_PLASTIC_SMD:SOD-123F, symbol 002_Basic_SingleSemiconductor:002_Diode_Schottky
- added D3: DS120W, 002_GN_TWO-PIN_PLASTIC_SMD:SOD-123F, symbol 002_Basic_SingleSemiconductor:002_Diode_Schottky
- added L1: 1uH, 008_GN_POWER-CHOKE_SMD:MC-2520, symbol 001_Basic_PassiveComponents:202_PowerChoke
- added R1: 100R, 001_GN_RCL_SMD:R0603(1608M), symbol 001_Basic_PassiveComponents:001_Resistor
- added R5: RL1210A680K, 001_GN_RCL_SMD:R1210(3225M), symbol 001_Basic_PassiveComponents:003_MetalOxideVaristors
- C11: renamed from C5; value 100uF -> 120uF
- C9: renamed from C4; value 12nF -> 1nF
- D5: renamed from D4; footprint 102_SP_POWER_DIODE_SMD:TO-277A -> 102_SP_POWER_DIODE_SMD:TO-277B
- D6: renamed from D3; footprint 102_SP_POWER_DIODE_SMD:TO-277A -> 102_SP_POWER_DIODE_SMD:TO-277B
- Q1: value HSBA20N15S -> HY1420C2
- renumbered C2 to C1, C1 to C10, C7 to C2, C9 to C8, D1 to D2, D2 to D4, R6 to R10, R1 to R2, R2 to R3, R8 to R6, R14 to R7, R10 to R8, R3 to R9, U2 to U1
Connections:
- net GND: now also C4.2, C5.2, C6.2, C7.2, L1.2, R5.1
- net GNDPWR: now also C12.2, C13.2, C14.2, C15.2, C16.2, C17.2, C18.2, C19.2
- net VBUS: now also C9.2, D2.1 (Cathode), C4.1, C5.1, C6.1, C7.1, R1.2, R5.2; no longer C2.1, C9.1, D2.2 (Anode), R2.1, U1.2 (Vin)
- net VDC: now also C12.1, C13.1, C14.1, C15.1, C16.1, C17.1, C18.1, C19.1
- net Vdrive: no longer C10.1, D4.1 (Cathode)
- new net: C9.1, D2.2 (Anode), D3.1 (Cathode)
- new net: D3.2 (Anode), L1.1
- new net: D1.2 (Anode), R1.1
- new net VDD: C10.1, C2.1, D1.1 (Cathode), D4.1 (Cathode), R2.1, U1.2 (Vin)
Other:
- moved on the sheet: C1, C10, C11, C2, C3, C8, C9, D2, D4, D5, D6, P1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

Commit message: Daily update
Parts:
- added R11: 2.2k, 001_GN_RCL_SMD:R1206(3216M), symbol 001_Basic_PassiveComponents:001_Resistor
Connections:
- net GNDPWR: now also R11.2
- net VDC: now also R11.1
Changed lines of the file:
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@@
+    (stroke (width 0) (type default))
+  )
+  (wire (pts (xy 271.78 55.88) (xy 264.16 55.88))
     (stroke (width 0) (type default))
   )
@@
     (stroke (width 0) (type default))
   )
+  (wire (pts (xy 271.78 73.66) (xy 271.78 101.6))
+    (stroke (width 0) (type default))
+  )
   (wire (pts (xy 218.44 55.88) (xy 210.82 55.88))
     (stroke (width 0) (type default))
@@
   )
   (wire (pts (xy 50.8 116.84) (xy 50.8 124.46))
+    (stroke (width 0) (type default))
+  )
+  (wire (pts (xy 271.78 63.5) (xy 271.78 55.88))
     (stroke (width 0) (type default))
   )
@@
         (path "/cc6fc110-a325-4469-a6c1-4bb061f00d5b"
           (reference "C17") (unit 1)
+        )
+      )
+    )
+  )
+  (symbol (lib_id "001_Basic_PassiveComponents:001_Resistor") (at 271.78 68.58 270) (unit 1)
+    (in_bom yes) (on_board yes) (dnp no) (fields_autoplaced)
+    (property "Reference" "R11" (at 274.32 67.31 90)
+      (effects (font (size 1.27 1.27)) (justify left))
+    )
+    (property "Value" "2.2k" (at 274.32 69.85 90)
+      (effects (font (size 1.27 1.27)) (justify left))
+    )
+    (property "Footprint" "001_GN_RCL_SMD:R1206(3216M)" (at 276.86 68.58 0)
+      (effects (font (size 1.27 1.27)) hide)
+    )
+    (property "Datasheet" "" (at 275.59 64.77 0)
+      (effects (font (size 1.27 1.27)) hide)
+    )
+    (property "Symbol type" "Alternate Source" (at 279.4 68.58 0)
+      (effects (font (size 1.27 1.27)) hide)
+    )
+    (pin "1")
+    (pin "2")
+    (instances
+      (project "Flyback_STD"
+        (path "/cc6fc110-a325-4469-a6c1-4bb061f00d5b"
+          (reference "R11") (unit 1)
         )
       )
@@
         )
       )
+    )
+  )
+  (symbol (lib_id "power:GNDPWR") (at 271.78 101.6 0) (unit 1)
+    (in_bom yes) (on_board yes) (dnp no) (fields_autoplaced)
+    (property "Reference" "#PWR038" (at 271.78 106.68 0)
+      (effects (font (size 1.27 1.27)) hide)
+    )
+    (property "Value" "GNDPWR" (at 271.78 106.68 0)
+      (effects (font (size 1.27 1.27)))
+    )
+    (property "Footprint" "" (at 271.78 102.87 0)
+      (effects (font (size 1.27 1.27)) hide)
+    )
+    (property "Datasheet" "" (at 271.78 102.87 0)
+      (effects (font (size 1.27 1.27)) hide)
+    )
+    (pin "1")
+    (instances
+      (project "Flyback_STD"
+        (path "/cc6fc110-a325-4469-a6c1-4bb061f00d5b"
+          (reference "#PWR038") (unit 1)
+        )
+      )

Commit message: Create new layout
Parts:
- L1: value 1uH -> 10uH
- R9: value 36k -> 33k
Changed lines of the file:
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@@
       (effects (font (size 1.27 1.27)) (justify left))
     )
-    (property "Value" "1uH" (at 143.51 103.505 90)
+    (property "Value" "10uH" (at 143.51 103.505 90)
       (effects (font (size 1.27 1.27)) (justify left))
     )
@@
       (effects (font (size 1.27 1.27)) (justify left))
     )
-    (property "Value" "36k" (at 157.48 103.505 90)
-      (effects (font (size 1.27 1.27)) (justify left))
-    )
+    (property "Value" "33k" (at 157.48 103.505 90)
+      (effects (font (size 1.27 1.27)) (justify left))
+    )

Commit message: Nightly update
Parts:
- added Q2: HSBB0012, 103_SP_POWER_TRANSISTOR_SMD:SON-FET_3333, symbol 202_Power_Transistor:001_MOSFET_N-ch
Connections:
- net CS: now also Q2.S (Source)
- net GT: now also Q2.G (Gate)
- net VBUS: now also Q2.D (Drain)
Other:
- moved on the sheet: C9
Changed lines of the file:
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@@
   (junction (at 124.46 55.88) (diameter 0) (color 0 0 0 0)
   )
-  (junction (at 162.56 78.74) (diameter 0) (color 0 0 0 0)
+  (junction (at 142.24 71.12) (diameter 0) (color 0 0 0 0)
   )
   (junction (at 218.44 55.88) (diameter 0) (color 0 0 0 0)
@@
   (junction (at 50.8 91.44) (diameter 0) (color 0 0 0 0)
   )
+  (junction (at 162.56 76.2) (diameter 0) (color 0 0 0 0)
+  )
   (junction (at 142.24 55.88) (diameter 0) (color 0 0 0 0)
   )
@@
   (junction (at 233.68 55.88) (diameter 0) (color 0 0 0 0)
   )
-  (junction (at 142.24 73.66) (diameter 0) (color 0 0 0 0)
-  )
   (junction (at 114.3 177.8) (diameter 0) (color 0 0 0 0)
   )
@@
   (junction (at 116.84 104.14) (diameter 0) (color 0 0 0 0)
   )
+  (junction (at 132.08 76.2) (diameter 0) (color 0 0 0 0)
+  )
   (junction (at 256.54 55.88) (diameter 0) (color 0 0 0 0)
   )
@@
   )
   (no_connect (at 96.52 114.3))
+  (wire (pts (xy 132.08 76.2) (xy 162.56 76.2))
+    (stroke (width 0) (type default))
+  )
   (wire (pts (xy 58.42 63.5) (xy 58.42 66.04))
     (stroke (width 0) (type default))
@@
     (stroke (width 0) (type default))
   )
-  (wire (pts (xy 157.48 73.66) (xy 162.56 73.66))
+  (wire (pts (xy 160.02 71.12) (xy 162.56 71.12))
     (stroke (width 0) (type default))
   )
@@
     (stroke (width 0) (type default))
   )
-  (wire (pts (xy 142.24 68.58) (xy 142.24 73.66))
+  (wire (pts (xy 142.24 68.58) (xy 142.24 71.12))
     (stroke (width 0) (type default))
   )
@@
     (stroke (width 0) (type default))
   )
-  (wire (pts (xy 142.24 73.66) (xy 142.24 83.82))
+  (wire (pts (xy 142.24 71.12) (xy 142.24 83.82))
     (stroke (width 0) (type default))
   )
@@
     (stroke (width 0) (type default))
   )
-  (wire (pts (xy 162.56 78.74) (xy 175.26 78.74))
+  (wire (pts (xy 162.56 76.2) (xy 175.26 76.2))
+    (stroke (width 0) (type default))
+  )
+  (wire (pts (xy 127 81.28) (xy 116.84 81.28))
     (stroke (width 0) (type default))
   )
@@
     (stroke (width 0) (type default))
   )
+  (wire (pts (xy 132.08 104.14) (xy 124.46 104.14))
+    (stroke (width 0) (type default))
+  )
   (wire (pts (xy 38.1 116.84) (xy 38.1 124.46))
     (stroke (width 0) (type default))
@@
     (stroke (width 0) (type default))
   )
-  (wire (pts (xy 124.46 78.74) (xy 124.46 83.82))
-    (stroke (width 0) (type default))
-  )
-  (wire (pts (xy 175.26 78.74) (xy 175.26 55.88))
+  (wire (pts (xy 124.46 76.2) (xy 124.46 83.82))
+    (stroke (width 0) (type default))
+  )
+  (wire (pts (xy 175.26 76.2) (xy 175.26 55.88))
     (stroke (width 0) (type default))
   )
@@
     (stroke (width 0) (type default))
   )
+  (wire (pts (xy 116.84 81.28) (xy 116.84 88.9))
+    (stroke (width 0) (type default))
+  )
   (wire (pts (xy 58.42 76.2) (xy 58.42 78.74))
     (stroke (width 0) (type default))
@@
     (stroke (width 0) (type default))
   )
+  (wire (pts (xy 132.08 86.36) (xy 132.08 104.14))
+    (stroke (width 0) (type default))
+  )
   (wire (pts (xy 73.66 114.3) (xy 76.2 114.3))
     (stroke (width 0) (type default))
@@
     (stroke (width 0) (type default))
   )
-  (wire (pts (xy 142.24 73.66) (xy 147.32 73.66))
-    (stroke (width 0) (type default))
-  )
-  (wire (pts (xy 124.46 78.74) (xy 162.56 78.74))
+  (wire (pts (xy 142.24 71.12) (xy 149.86 71.12))
+    (stroke (width 0) (type default))
+  )
+  (wire (pts (xy 124.46 76.2) (xy 132.08 76.2))
     (stroke (width 0) (type default))
   )
@@
     (stroke (width 0) (type default))
   )
-  (wire (pts (xy 162.56 73.66) (xy 162.56 78.74))
+  (wire (pts (xy 162.56 71.12) (xy 162.56 76.2))
     (stroke (width 0) (type default))
   )
@@
     )
   )
-  (symbol (lib_id "001_Basic_PassiveComponents:101_Capacitor") (at 152.4 73.66 0) (unit 1)
-    (in_bom yes) (on_board yes) (dnp no) (fields_autoplaced)
-    (property "Reference" "C9" (at 152.4 68.58 0)
-      (effects (font (size 1.27 1.27)))
-    )
-    (property "Value" "1nF" (at 152.4 71.12 0)
-      (effects (font (size 1.27 1.27)))
-    )
-    (property "Footprint" "001_GN_RCL_SMD:C0805(2012M)" (at 152.4 68.58 0)
-      (effects (font (size 1.27 1.27)) hide)
-    )
-    (property "Datasheet" "" (at 152.4 73.66 0)
-      (effects (font (size 1.27 1.27)) hide)
-    )
-    (property "Symbol type" "Alternate Source" (at 152.4 66.04 0)
+  (symbol (lib_id "001_Basic_PassiveComponents:101_Capacitor") (at 154.94 71.12 0) (unit 1)
+    (in_bom yes) (on_board yes) (dnp no) (fields_autoplaced)
+    (property "Reference" "C9" (at 154.94 66.04 0)
+      (effects (font (size 1.27 1.27)))
+    )
+    (property "Value" "1nF" (at 154.94 68.58 0)
+      (effects (font (size 1.27 1.27)))
+    )
+    (property "Footprint" "001_GN_RCL_SMD:C0805(2012M)" (at 154.94 66.04 0)
+      (effects (font (size 1.27 1.27)) hide)
+    )
+    (property "Datasheet" "" (at 154.94 71.12 0)
+      (effects (font (size 1.27 1.27)) hide)
+    )
+    (property "Symbol type" "Alternate Source" (at 154.94 63.5 0)
       (effects (font (size 1.27 1.27)) hide)
     )
@@
         )
       )
+    )
+  )
+  (symbol (lib_id "202_Power_Transistor:001_MOSFET_N-ch") (at 132.08 81.28 0) (unit 1)
+    (in_bom yes) (on_board yes) (dnp no) (fields_autoplaced)
+    (property "Reference" "Q2" (at 134.62 80.01 0)
+      (effects (font (size 1.27 1.27)) (justify left))
+    )
+    (property "Value" "HSBB0012" (at 134.62 82.55 0)
+      (effects (font (size 1.27 1.27)) (justify left))
+    )
+    (property "Footprint" "103_SP_POWER_TRANSISTOR_SMD:SON-FET_3333" (at 153.67 77.47 0)
+      (effects (font (size 1.27 1.27)) hide)
+    )
+    (property "Datasheet" "" (at 132.715 81.28 0)
+      (effects (font (size 1.27 1.27)) hide)
+    )
+    (property "Symbol type" "Alternate Source" (at 143.51 77.47 0)
+      (effects (font (size 1.27 1.27)) hide)
+    )
+    (property "LCSC" "C701044" (at 132.08 81.28 0)
+      (effects (font (size 1.27 1.27)) hide)
+    )
+    (pin "D")
+    (pin "G")
+    (pin "S")
+    (instances
+      (project "Flyback_STD"
+        (path "/cc6fc110-a325-4469-a6c1-4bb061f00d5b"
+          (reference "Q2") (unit 1)
+        )
+      )
