File: Flyback_STD.kicad_sch (KiCad schematic)
At the start: 44 parts, among them P1 VIN, P2 GND, P3 VOUT, P4 PGND, Q1 HY1420C2, Q2 HSBB0012, U1 VPC2188B

Commit message: Remake project
Parts:
- removed D5, D6: SB2080L, 102_SP_POWER_DIODE_SMD:TO-277B, symbol 201_Power_Diode:002_Diode_Schottky
- added C20: 10nF, 001_GN_RCL_SMD:C0603(1608M), symbol 001_Basic_PassiveComponents:101_Capacitor
- added D7: MM3Z10, 002_GN_TWO-PIN_PLASTIC_SMD:SOD-123, symbol 002_Basic_SingleSemiconductor:003_Diode_Zener
- added PC1: OR-3H7B-TP-G, symbol Flyback:PC-4
- added Q3: MMBT3904, 003_GN_SMALL-SEMI_SMD:SOT-323, symbol 002_Basic_SingleSemiconductor:101_BJT_NPN
- added R12: 10k, 001_GN_RCL_SMD:R0603(1608M), symbol 001_Basic_PassiveComponents:001_Resistor
- added T1: TRF-9_2-2-A1, symbol Flyback:TRF-9_2-2-A1
- added U2: DS8606-A1A3, 004_GN_MIDDLE-SEMI_SMD:SOT-89_4525, symbol 203_Power_LDO:DS8606-A1A3
- added U3: TL431, 003_GN_SMALL-SEMI_SMD:SOT-23, symbol 103_IntegratedCircuit_Reference:TL431
- C2: value 100nF -> 10uF; footprint 001_GN_RCL_SMD:C0603(1608M) -> 001_GN_RCL_SMD:C0805(2012M)
- C9: value 1nF -> 3.3nF
- D1: value DS110W -> 1N5819; footprint 002_GN_TWO-PIN_PLASTIC_SMD:SOD-123F -> 002_GN_TWO-PIN_PLASTIC_SMD:SOD-323
- D2, D3: value DS120W -> DS220W
- D4: value DS110W -> DS220W
- L1: value 10uH -> 22uH
- Q1: value HY1420C2 -> HY1420P; footprint 103_SP_POWER_TRANSISTOR_SMD:SON-FET_6050 -> 153_SP_POWER_TRANSISTOR_THD:TO247-3_HR1620
- Q2: value HSBB0012 -> HY1420P; footprint 103_SP_POWER_TRANSISTOR_SMD:SON-FET_3333 -> (none); LCSC C701044 -> (none)
- R1: value 100R -> 2kR
- R10: value 3.9k -> 39k
- R11: value 2.2k -> 10k
- R6: value 2.2R -> 10R
- R9: value 33k -> 10k
Connections:
- net CS: no longer Q2.S (Source)
- net GND: now also D7.2 (Anode), PC1.3 (Emitter), R12.2, T1.2, U2.2 (GND), U3.3 (A); no longer D4.2 (Anode), R10.2, R9.1
- net GNDPWR: now also Q2.S (Source)
- net GT: now also D1.2 (Anode); no longer Q2.G (Gate)
- net GT_U: now also D1.1 (Cathode)
- net VBUS: now also R2.1, Q3.3 (Collector), T1.1; no longer C9.2, Q1.D (Drain), Q2.D (Drain)
- net VDC: now also R10.1, R9.1, PC1.1 (Anode), T1.8
- net Vdrive: now also C2.1, U2.1 (Vout)
- net COMP: now reaches U1.1 (COM)
- net COMP: now also PC1.4 (Collector)
- net at R1.1: now also D7.1 (Cathode), Q3.1 (Base); no longer D1.2 (Anode)
- removed net VDD: C10.1, C2.1, D1.1 (Cathode), D4.1 (Cathode), R2.1, U1.2 (Vin)
- new net: C10.1, D4.1 (Cathode), U2.3 (Vin)
- new net: D4.2 (Anode), T1.3
- new net: C9.2, Q1.D (Drain), T1.4
- new net: Q2.D (Drain), T1.6
- new net: C20.2, PC1.2 (Cathode), R9.2, U3.2 (K)
- new net REF_2V5: C20.1, R10.2, R12.1, U3.1 (Ref)
- new net Vin: Q3.2 (Emitter), U1.2 (Vin)
- now unconnected: U1.10 (FB)
- no-connect marks 1 -> 3
Other:
- moved on the sheet: C1, C10, C11, C12, C13, C14, C15, C16, C17, C18, C19, C3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
