File: Coil_1p75/Coil_1p75.kicad_pcb (KiCad board)
At the start: 2 copper layers, 0 parts

Commit message: Update coil
Routing:
- net (no net): vias 0 -> 6
Other:
- board outline added: 22.5 x 22 mm

Commit message: Daily update
Routing:
- net (no net): track 0.00 -> 118.7 mm, vias 6 -> 18
Changed lines of the file:
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@@
     )
     (stroke (width 0) (type solid)) (fill solid) (layer "B.Cu"))
+  (gr_line (start 137.375 100) (end 137.625 100)
+    (stroke (width 0.15) (type default)) (layer "Dwgs.User"))
   (gr_line (start 87.5 87.5) (end 112.5 112.5)
     (stroke (width 0.1) (type default)) (layer "Dwgs.User"))
   (gr_line (start 87.5 112.5) (end 112.5 87.5)
     (stroke (width 0.1) (type default)) (layer "Dwgs.User"))
+  (gr_line (start 137.5 99.875) (end 137.5 100.125)
+    (stroke (width 0.15) (type default)) (layer "Dwgs.User"))
   (gr_arc (start 91.953219 92.5) (mid 100 89) (end 108.046781 92.5)
     (stroke (width 0.1) (type default)) (layer "Edge.Cuts"))
@@
   (gr_circle locked (center 100 100) (end 106 100)
     (stroke (width 0.2) (type solid)) (fill solid) (layer "F.Fab"))
+  (segment (start 130.156332 98.261395) (end 129.386625 99.031101) (width 2.05) (layer "F.Cu") (net 0))
+  (segment (start 124 96.55) (end 124 93.75) (width 2.05) (layer "F.Cu") (net 0))
+  (segment (start 122.600952 99.350951) (end 121.625 98.375) (width 2.05) (layer "F.Cu") (net 0))
+  (segment (start 126.052295 98.05) (end 125.5 98.05) (width 2.05) (layer "F.Cu") (net 0))
+  (segment (start 128.6751 96.028235) (end 127.078335 97.625) (width 2.05) (layer "F.Cu") (net 0))
+  (segment (start 125.625 100.5) (end 125.375 100.5) (width 2.05) (layer "F.Cu") (net 0))
+  (segment (start 128.006575 102.362836) (end 128.561466 103.702462) (width 2.05) (layer "F.Cu") (net 0))
+  (segment (start 130.09555 101.591868) (end 130.617097 102.850992) (width 2.05) (layer "F.Cu") (net 0))
+  (segment (start 130.617097 97.149008) (end 130.156332 98.261395) (width 2.05) (layer "F.Cu") (net 0))
+  (via (at 130.25 100.5) (size 0.5) (drill 0.3) (layers "F.Cu" "B.Cu") (net 0))
+  (via (at 125.75 100.5) (size 0.5) (drill 0.3) (layers "F.Cu" "B.Cu") (net 0))
   (via (at 91.25 101.75) (size 0.6) (drill 0.3) (layers "F.Cu" "B.Cu") (net 0))
+  (via (at 129.625 100.625) (size 0.5) (drill 0.3) (layers "F.Cu" "B.Cu") (net 0))
   (via (at 90.5 101.625) (size 0.6) (drill 0.3) (layers "F.Cu" "B.Cu") (net 0))
+  (via (at 125.5 101.125) (size 0.5) (drill 0.3) (layers "F.Cu" "B.Cu") (net 0))
+  (via (at 125.5 99.875) (size 0.5) (drill 0.3) (layers "F.Cu" "B.Cu") (net 0))
   (via (at 91.875 101.25) (size 0.6) (drill 0.3) (layers "F.Cu" "B.Cu") (net 0))
+  (via (at 126.375 100.500001) (size 0.5) (drill 0.3) (layers "F.Cu" "B.Cu") (net 0))
+  (via (at 126.124999 101.125) (size 0.5) (drill 0.3) (layers "F.Cu" "B.Cu") (net 0))
+  (via (at 126.125 99.875) (size 0.5) (drill 0.3) (layers "F.Cu" "B.Cu") (net 0))
+  (via (at 130.375 101.625) (size 0.5) (drill 0.3) (layers "F.Cu" "B.Cu") (net 0))
+  (via (at 129.75 101.75) (size 0.5) (drill 0.3) (layers "F.Cu" "B.Cu") (net 0))
   (via (at 93.25 100.875) (size 0.6) (drill 0.3) (layers "F.Cu" "B.Cu") (net 0))
   (via (at 89.875 102.125) (size 0.6) (drill 0.3) (layers "F.Cu" "B.Cu") (net 0))
+  (via (at 129.375 101.25) (size 0.5) (drill 0.3) (layers "F.Cu" "B.Cu") (net 0))
   (via (at 92.625 101.375) (size 0.6) (drill 0.3) (layers "F.Cu" "B.Cu") (net 0))
+  (via (at 130 101.125) (size 0.5) (drill 0.3) (layers "F.Cu" "B.Cu") (net 0))
+  (arc (start 146.438534 96.297538) (mid 141.202462 91.061466) (end 133.797538 91.061466) (width 2.05) (layer "F.Cu") (net 0))
+  (arc (start 133.797538 91.061466) (mid 130.762848 93.056197) (end 128.6751 96.028235) (width 2.05) (layer "F.Cu") (net 0))
+  (arc (start 125.5 98.05) (mid 124.43934 97.61066) (end 124 96.55) (width 2.05) (layer "F.Cu") (net 0))
+  (arc (start 134.649008 93.117097) (mid 132.232054 94.732054) (end 130.617097 97.149008) (width 2.05) (layer "F.Cu") (net 0))
+  (arc (start 128.561466 103.702462) (mid 133.797538 108.938534) (end 141.202462 108.938534) (width 2.05) (layer "F.Cu") (net 0))
+  (arc (start 144.382903 97.149008) (mid 140.350992 93.117097) (end 134.649008 93.117097) (width 2.05) (layer "F.Cu") (net 0))
+  (arc (start 129.386625 99.031101) (mid 128.006575 100.411151) (end 128.006575 102.362836) (width 2.05) (layer "F.Cu") (net 0))
+  (arc (start 141.202462 108.938534) (mid 146.438534 103.702462) (end 146.438534 96.297538) (width 2.05) (layer "F.Cu") (net 0))
+  (arc (start 125.375 100.5) (mid 123.873696 100.201372) (end 122.600952 99.350951) (width 2.05) (layer "F.Cu") (net 0))
+  (arc (start 130.09555 101.199897) (mid 130.056567 101.395883) (end 130.09555 101.591868) (width 2.05) (layer "F.Cu") (net 0))
+  (arc (start 127.078335 97.625) (mid 126.607584 97.939546) (end 126.052295 98.05) (width 2.05) (layer "F.Cu") (net 0))
+  (arc (start 130.617097 102.850992) (mid 134.640103 106.873998) (end 140.350992 106.882903) (width 2.05) (layer "F.Cu") (net 0))
+  (arc (start 140.350992 106.882903) (mid 144.382903 102.838398) (end 144.382903 97.149008) (width 2.05) (layer "F.Cu") (net 0))
+  (segment (start 126 100.5) (end 128.216117 100.5) (width 2.05) (layer "B.Cu") (net 0))
+  (arc (start 128.216117 100.5) (mid 129.032718 100.662432) (end 129.725 101.125) (width 2.05) (layer "B.Cu") (net 0))
 )
